File: Ruler_Electronic.sch (KiCad schematic (older format))
At the start: 58 parts, among them J1 USB_OTG, J2 CONN_01X03, J3 CONN_01X02, J4 CONN_01X02, SW1 SW_Push, SW2 SW_Push, SW3 SW_Push, SW4 SW_Push, SW5 SW_Push, U1 USBLC6-2SC6, U2 ATMEGA8U2-AU, U3 MCP2515-E/ST, U4 MCP2561-E/SN, Y1 ABM8-16.000MHZ-B2-T, Y2 ABM8-20.000MHZ-B2-T

Commit message: finished layout
Parts:
- removed SW1, SW2, SW3, SW4, SW5: SW_Push, Buttons_Switches_SMD:SW_SPST_EVPBF, symbol SW_Push
- added ME1: LOGO, logo:bytewerk_logo_15x13mm, symbol LOGO
- added R22, R23, R24, R25, R26: 560R, Resistors_SMD:R_0603_HandSoldering, symbol R
- added S1, S2, S3, S4, S5: Marquardt_3006.2115, shlib-switches:Marquardt_3006.2xxx, symbol Marquardt_3006.2115
- L1, L2, L3: value L -> WE_742863147
- R12, R13: value 1k -> 560R
- R14, R15, R16, R18, R8: value R -> 10k
Connections:
- net GND: now also S1.2, S1.K, S2.2, S2.K, S3.2, S3.K, S4.2, S4.K, S5.2, S5.K
- net at R18.2, U2.10 ((INT5/AIN3)PD4): now also S5.1
- net at R16.2, U2.11 ((XCK/AIN4/PCINT12)PD5): now also S4.1
- net at R15.2, U2.12 ((~RTS~/AIN5/INT6)PD6): now also S3.1
- net at R14.2, U2.13 ((~CTS~/~HWB~/AIN6/T0/INT7)PD7): now also S2.1
- net at U2.21 ((PCINT7/OC.0A/OC.1C)PB7): now also R26.1
- net at U2.22 ((INT4/ICP1/CLK0)PC7): now also R22.1
- net at U2.23 ((OC.1A/PCINT8)PC6): now also R23.1
- net at U2.25 ((PCINT9/OC.1B)PC5): now also R24.1
- net at U2.26 ((PCINT10)PC4): now also R25.1
- net at R8.2, U2.5 ((PCINT11/AIN2)PC2): now also S1.1
- new net: R22.2, S1.A
- new net: R23.2, S2.A
- new net: R24.2, S3.A
- new net: R25.2, S4.A
- new net: R26.2, S5.A
- no-connect marks 8 -> 7
