File: Ruler_Electronic.kicad_pcb (KiCad board)
At the start: 2 copper layers, 307 x 40 mm, 59 parts, among them J1 USB_OTG, J2 CONN_01X03, J3 CONN_01X02, J4 CONN_01X02, SW1 SW_Push, SW2 SW_Push, SW3 SW_Push, SW4 SW_Push, SW5 SW_Push, U1 USBLC6-2SC6, U2 ATMEGA8U2-AU, U3 MCP2515-E/ST, U4 MCP2561-E/SN, Y1 ABM8-16.000MHZ-B2-T, Y2 ABM8-20.000MHZ-B2-T

Commit message: blubb
Signed-off-by: stephan <stephan.hueltl@gmx.de>
Parts:
- removed G***: LOGO, logo:LOGO
- removed SW1, SW2, SW3, SW4, SW5: SW_Push, Buttons_Switches_SMD:SW_SPST_EVPBF
- added ME1: LOGO, logo:bytewerk_logo_15x13mm, F.Cu at (326.0, 122.2)
- added R22: 560R, Resistors_SMD:R_0603_HandSoldering, F.Cu at (202.5, 130.0)
- added R23: 560R, Resistors_SMD:R_0603_HandSoldering, F.Cu at (331.6, 132.5)
- added R24: 560R, Resistors_SMD:R_0603_HandSoldering, F.Cu at (300.0, 130.0)
- added R25: 560R, Resistors_SMD:R_0603_HandSoldering, F.Cu at (267.5, 130.0)
- added R26: 560R, Resistors_SMD:R_0603_HandSoldering, F.Cu at (235.0, 130.0)
- added S1: Marquardt_3006.2115, shlib-switches:Marquardt_3006.2xxx, F.Cu at (212.5, 132.5)
- added S2: Marquardt_3006.2115, shlib-switches:Marquardt_3006.2xxx, F.Cu at (342.5, 132.5)
- added S3: Marquardt_3006.2115, shlib-switches:Marquardt_3006.2xxx, F.Cu at (310.0, 132.5)
- added S4: Marquardt_3006.2115, shlib-switches:Marquardt_3006.2xxx, F.Cu at (277.5, 132.5)
- added S5: Marquardt_3006.2115, shlib-switches:Marquardt_3006.2xxx, F.Cu at (245.0, 132.5)
- FL1: footprint Inductors_SMD_self:L_Murata_DLP11S -> Inductors_SMD_self:DLP11S
- L1, L2, L3: value L -> WE_742863147
- R12, R13: value 1k -> 560R
- R14, R15, R16, R18, R8: value R -> 10k
- moved R17 55.1 mm to (172.1, 116.2), turned to 180 degrees
- moved C11 3.00 mm to (137.1, 119.3)
- moved C12 3.00 mm to (137.1, 116.9)
- moved R11 3.00 mm to (133.0, 121.3)
- moved Y2 3.00 mm to (133.0, 118.0)
- moved J1 1.75 mm to (54.2, 125.5)
- moved C13 0.50 mm to (125.3, 125.3)
- turned FL1 to 0 degrees
Connections:
- U2 pad 21: (no net) -> Net-(R26-Pad1)
- U2 pad 22: (no net) -> Net-(R22-Pad1)
- U2 pad 23: (no net) -> Net-(R23-Pad1)
- U2 pad 25: (no net) -> Net-(R24-Pad1)
- U2 pad 26: (no net) -> Net-(R25-Pad1)
Routing:
- net Net-(R23-Pad1): track 0.00 -> 281.4 mm, vias 0 -> 2
- net Net-(R24-Pad1): track 0.00 -> 224.3 mm, vias 0 -> 2
- net Net-(R25-Pad1): track 0.00 -> 193.6 mm, vias 0 -> 2
- net Net-(R26-Pad1): track 0.00 -> 168.7 mm, vias 0 -> 2
- net Net-(R14-Pad2): track 104.4 -> 254.0 mm
- net Net-(R22-Pad1): track 0.00 -> 149.0 mm, vias 0 -> 2
- net Net-(R15-Pad2): track 103.9 -> 217.8 mm
- net Net-(R16-Pad2): track 103.8 -> 184.5 mm
- net Net-(R18-Pad2): track 103.4 -> 151.0 mm
- net +5V: track 50.4 -> 33.2 mm, vias 10 -> 11
- net Net-(R8-Pad2): track 115.3 -> 127.2 mm
- net Net-(C1-Pad1): track 27.4 -> 34.4 mm
- net Net-(R23-Pad2): track 0.00 -> 6.81 mm
- net Net-(D1-Pad1): track 75.2 -> 79.3 mm
- net Net-(R26-Pad2): track 0.00 -> 3.90 mm
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Other:
- net class Default: clearance 0.2 -> 0.199
- rule trace_clearance: 0.2 -> 0.199

Commit message: change in layout and new logo
Parts:
- removed ME1: LOGO, logo:bytewerk_logo_15x13mm
- added G***: LOGO, logo:bytewerk_logo_25x22mm, F.Cu at (342.2, 127.0)
- moved S2 28.5 mm to (314.0, 132.5)
- moved R23 27.4 mm to (304.4, 130.0)
- moved R24 21.6 mm to (278.4, 130.0)
- moved S3 21.0 mm to (289.0, 132.5)
- moved R25 13.8 mm to (253.7, 130.0)
- moved S4 13.5 mm to (264.0, 132.5)
- moved R14 9.25 mm to (183.9, 120.2)
- moved R15 9.25 mm to (183.9, 122.2)
- moved R16 9.25 mm to (183.9, 124.0)
- moved R18 9.25 mm to (183.9, 125.8)
- moved R8 9.25 mm to (183.9, 127.5)
- moved R26 6.15 mm to (228.8, 130.0)
- moved S5 6.00 mm to (239.0, 132.5)
- moved S1 1.50 mm to (214.0, 132.5)
- moved R22 0.90 mm to (203.4, 130.0)
Routing:
- net Net-(R23-Pad1): track 281.4 -> 250.1 mm
- net Net-(R14-Pad2): track 254.0 -> 226.1 mm
- net Net-(R24-Pad1): track 224.3 -> 202.7 mm
- net Net-(R15-Pad2): track 217.8 -> 196.8 mm
- net Net-(R25-Pad1): track 193.6 -> 179.8 mm
- net Net-(R16-Pad2): track 184.5 -> 171.0 mm
- net Net-(R22-Pad1): track 149.0 -> 142.2 mm
- net Net-(R26-Pad1): track 168.7 -> 162.5 mm
- net Net-(R18-Pad2): track 151.0 -> 145.0 mm
- net Net-(R23-Pad2): track 6.81 -> 3.50 mm
- net Net-(R8-Pad2): track 127.2 -> 128.9 mm
- net Net-(R24-Pad2): track 3.90 -> 4.55 mm
- net Net-(R22-Pad2): track 3.90 -> 4.50 mm
Other:
- rule trace_min: 0.2 -> 0.199
